File: design_blocks/TPSM843321_3V3.kicad_block/TPSM843321_3V3.kicad_pcb (KiCad board)
At the start: 6 copper layers, 25 parts, among them J2002 RFShield_TwoPieces_Frame_W31.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, J2003 RFShield_TwoPieces_Cover_W31.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, U2003 TPSM843321RCJR

Commit message: Added lots of block design
Parts:
- removed J2002: RFShield_TwoPieces_Frame_W31.2mm_L30mm_H5mm, gwd_library:MS312-10
- removed J2003: RFShield_TwoPieces_Cover_W31.2mm_L30mm_H5mm, gwd_library:MS312-10C
- added SH2102: RFShield_TwoPieces_Frame_W31.2mm_L30mm_H5mm, gwd_library:MS312-10, F.Cu at (192.1, 129.7)
- added SH2103: RFShield_TwoPieces_Cover_W31.2mm_L30mm_H5mm, gwd_library:MS312-10C, F.Cu at (192.1, 129.7)
Connections:
- net /fpga/3.3V_PG renamed /fpga/PG
- net /fpga/Sys_PG renamed /fpga/EN
- R2036 pad 2: unconnected-(R2036-Pad2) -> GND
Routing:
- net Net-(U2003-EN): track 29.3 -> 0.00 mm
- net /fpga/PG: track 16.2 -> 0.00 mm, vias 2 -> 0
- net Net-(U2003-FB): track 11.1 -> 0.00 mm
- net /fpga/TPS_VOUT: track 4.89 -> 0.00 mm, vias 3 -> 0
- net Net-(U2003-RT_SYNC): track 4.36 -> 0.00 mm
- net Net-(U2003-MODE): track 3.83 -> 0.00 mm
- net GND: track 3.63 -> 0.00 mm, vias 118 -> 0
- net /fpga/VDD_3V3: vias 4 -> 0
- net /VDD_12V: vias 5 -> 0
- removed copper zone on F.Cu, net /VDD_12V
- removed copper zone on B.Cu, net /fpga/TPS_VIN
- removed copper zone on F.Cu, net /fpga/TPS_VIN
- removed copper zone on B.Cu, net /fpga/TPS_VOUT
- removed copper zone on F.Cu, net /fpga/TPS_VOUT
- removed copper zone on F.Cu, net /fpga/VDD_3V3
