File: design_blocks/TPSM843321_3V3.kicad_block/TPSM843321_3V3.kicad_sch (KiCad schematic)
At the start: 25 parts, among them J2002 RFShield_TwoPieces_Frame_W31.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, J2003 RFShield_TwoPieces_Cover_W31.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, U2003 TPSM843321RCJR

Commit message: Added lots of block design
Parts:
- renumbered J2002 to SH2102, J2003 to SH2103
Connections:
- net GND: now also R2036.2
- net 3.3V_PG renamed PG
- net Sys_PG renamed EN
Other:
- moved on the sheet: C2017, C2018, C2019, C2020, C2021, C2022, C2023, C2039, C2040, C2041, FB2003, FB2004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
